File: Projects/Client Name/My_ECS/Design/ECS/MOSTFET DRIVER.kicad_sch (KiCad schematic)
At the start: 0 parts

Commit message: MOSFET DRIVER Schematic done
Parts:
- added C18: 120p, symbol Device:C
- added C19, C27, C28, C29, C33, C34, C35, C36, C37, C38, C40, C41: 10u, symbol Device:C
- added C20: 6.8n, symbol Device:C
- added C21, C22, C23, C24, C26: 2u2, symbol Device:C
- added C25: 22n, symbol Device:C
- added C30, C31, C32: 220n, symbol Device:C
- added C39: 100n, symbol Device:C
- added D4: BAT60A, Diode_SMD:D_SOD-323, symbol Diode:BAT60A
- added D6: PMEG6020, Diode_SMD:Nexperia_CFP3_SOD-123W, symbol Diode:PMEG6020AELR
- added L1: 22u, symbol Device:L
- added R11: 205K, symbol Device:R
- added R12: 16K2, symbol Device:R
- added R13: 10K, symbol Device:R
- added R14: 1M, symbol Device:R
- added R15: 18K, symbol Device:R
- added R16, R18, R20, R22: 3K3, symbol Device:R
- added R17, R19, R21: 39K, symbol Device:R
- added U2: DRV8302DCAR, DCA56_6P35X3P61, symbol 2024-09-27_03-49-45:DRV8302DCAR
Connections:
- new net: C20.2, R12.1
- new net: C26.1, U2.27 (AVDD)
- new net +3V3: U2.24 (REF)
- new net +3v3: U2.9 (M_OC)
- new net +5V: D4.1 (K)
- new net +5V_DRV: C19.1, C40.1, C41.1, D4.2 (A), L1.2, R15.2
- new net +VDC: C27.1, C28.1, C29.1, C33.1, C34.1, C35.1, C36.1, C37.1, C38.1, U2.29 (PVDD1), U2.53 (PVDD2), U2.54 (PVDD2)
- new net BIAS: R14.1, U2.49 (BIAS)
- new net BR_SO1: U2.25 (SO1)
- new net BR_SO2: U2.26 (SO2)
- new net BST_A: C30.1, U2.48 (BST_A)
- new net BST_B: C31.1, U2.43 (BST_B)
- new net BST_BK: C39.1, U2.52 (BST_BK)
- new net BST_C: C32.1, U2.38 (BST_C)
- new net COMP: C18.2, R12.2, U2.2 (COMP)
- new net CP1: C25.1, U2.14 (CP1)
- new net CP2: C25.2, U2.15 (CP2)
- new net DC_CAL: U2.12 (DC_CAL)
- new net DTC: R13.2, U2.7 (DTC)
- new net DVDD: C21.1, C22.1, U2.11 (OC_ADJ), U2.23 (DVDD)
- new net EN_GATE: U2.16 (EN_GATE)
- new net FAULT: U2.6 (*FAULT)
- new net GND: C18.1, C19.2, C20.1, C21.2, C22.2, C23.2, C24.2, C26.2, C27.2, C28.2, C29.2, C33.2, C34.2, C35.2, C36.2, C37.2, C38.2, C40.2, C41.2, D6.2 (A), R11.1, R13.1, R14.2, R16.1, R18.1, R20.1, R22.1, U2.10 (GAIN), U2.28 (AGND), U2.57 (EPAD), U2.8 (M_PWM)
- new net GVDD: C23.1, C24.1, U2.13 (GVDD)
- new net H1: U2.17 (INH_A)
- new net H1_LOW: U2.44 (SL_A)
- new net H1_VS: C30.2, R21.2, U2.46 (SH_A)
- new net H2: U2.19 (INH_B)
- new net H2_LOW: U2.39 (SL_B)
- new net H2_VS: C31.2, R19.2, U2.41 (SH_B)
- new net H3: U2.21 (INH_C)
- new net H3_LOW: U2.34 (SL_C)
- new net H3_VS: C32.2, R17.2, U2.36 (SH_C)
- new net L1: U2.18 (INL_A)
- new net L2: U2.20 (INL_B)
- new net L3: U2.22 (INL_C)
- new net M_H1: U2.47 (GH_A)
- new net M_H2: U2.42 (GH_B)
- new net M_H3: U2.37 (GH_C)
- new net M_L1: U2.45 (GL_A)
- new net M_L2: U2.40 (GL_B)
- new net M_L3: U2.35 (GL_C)
- new net PH: C39.2, D6.1 (K), L1.1, U2.50 (PH), U2.51 (PH)
- new net RT_CLK: R11.2, U2.1 (RT_CLK)
- new net SENS1: R17.1, R18.2
- new net SENS2: R19.1, R20.2
- new net SENS3: R21.1, R22.2
- new net SN1: U2.33 (SN1)
- new net SN2: U2.31 (SN2)
- new net SP1: U2.32 (SP1)
- new net SP2: U2.30 (SP2)
- new net VSENSE: R15.1, R16.2, U2.3 (VSENSE)
Other:
- note added: "10u DECOUPLING PLACE AS CLOSE AS POSIBLE TO THE IC"
- note added: "BOOTSTRAP CAPs"
- note added: "BULK CAPACITANCE KEEP AS CLOSE AS POSIBLE TO THE IC AND TO THE DRIVER INPUT LOOP"
- note added: "Hx_VS"
- note added: "INPUT PORTS"
- note added: "KEEP AWAY FROM NOISE TRACKS AND COMPONENTS"
- note added: "MCU must sense the voltage at each phase"
- note added: "OUTPUT PORTS"
- note added: "SENSE 1 - PHASE 3"
- note added: "SENSE 2 - PHASE 1"
- note added: "[5] - MOSFET DRIVER"
